File: led_strip/led_strip.kicad_pcb (KiCad board)
At the start: 2 copper layers, 142.2 x 43.2 mm, 25 parts, among them J1 Conn_01x03_Socket

Commit message: init
Parts:
- LED1, LED10, LED11, LED12, LED13, LED14, LED15, LED16, LED17, LED18, LED19, LED2, LED20, LED21, LED22, LED23, LED24, LED3, LED4, LED5, LED6, LED7, LED8, LED9: footprint lib:LED_SK6812MINI-R -> sk6812:LED_SK6812MINI-R
